Commit message: with .gitignore

File: src/simble_box_bot/urdf/balance_bot.xacro (robot description, xacro)
@@ -25,10 +25,4 @@
         </inertial>
     </xacro:macro>
-    <!-- <link name="world"/> -->
-    <!-- <joint name="fixed_to_world" type="fixed">
-        <parent link="world"/>
-        <child link="base_link"/>
-        <origin xyz="0 0 0.4" rpy="0 0 0"/>
-    </joint> -->
     <link name="base_link">
         <visual>

Commit message: only simble_box controled by lqr

File: src/simble_box_bot/urdf/balance_bot.xacro (robot description, xacro)
@@ -63,5 +63,5 @@
             <child link="${prefix}_wheel"/>
             <origin xyz="0 ${reflect * (chassis_depth/2 + wheel_width/2 + 0.01)} -${chassis_height/2 + 0.02}" rpy="0 0 0"/>
-            <axis xyz="0 1 0"/> <limit effort="10.0" velocity="20.0"/> <dynamics damping="0.1" friction="0.1"/> </joint>
+            <axis xyz="0 1 0"/> <limit effort="3.0" velocity="70.0"/> <dynamics damping="0.01" friction="0.01"/> </joint>
         <transmission name="${prefix}_wheel_trans">
             <type>transmission_interface/SimpleTransmission</type>
@@ -96,5 +96,5 @@
             </geometry>
         </collision>
-        <xacro:box_inertial m="0.01" w="0.02" d="0.02" h="0.01"/>
+        <!-- <xacro:box_inertial m="0.01" w="0.02" d="0.02" h="0.01"/> -->
     </link>
     <joint name="imu_joint" type="fixed">
